File: hw_design/binary_watch/binary_watch.kicad_pcb (KiCad board)
At the start: 2 copper layers, 35.6 x 35.6 mm, 32 parts, among them J1 Conn_01x06, J2 Conn_02x03_Counter_Clockwise, SW1 SW_Push, U1 ATmega328P-AU, U2 MCP7940N-xMS, Y1 32.758kHz

Commit message: [update] Place PCB Components
Place all components on pcb layout to start routing.
Parts:
- C1, C2, C3, R1, R2, R3: moved to B.Cu
- moved C3 59.6 mm to (173.2, 91.8), turned to 135 degrees
- moved C2 56.4 mm to (176.8, 88.3), turned to 135 degrees
- moved C1 55.6 mm to (175.0, 90.1), turned to 135 degrees
- moved R2 32.3 mm to (194.8, 89.0), turned to 180 degrees
- moved R3 32.1 mm to (197.1, 91.6), turned to 180 degrees
- moved R1 16.8 mm to (198.6, 106.8), turned to 135 degrees
- moved C5 9.50 mm to (180.6, 87.0), turned to 180 degrees
- moved C4 9.24 mm to (190.0, 87.0), turned to 0 degrees
- moved J1 8.03 mm to (170.9, 100.5), turned to 180 degrees
- moved J2 1.80 mm to (194.6, 110.9)
- turned Y1 to 180 degrees
Connections:
- C3 pad 1: /VCC -> /RST
- C3 pad 2: GND -> Net-(C3-Pad2)
- J1 pad 1: Net-(J1-Pad1) -> Net-(C3-Pad2)

Commit message: [update] Schematic and PCB
Parts:
- moved J1 0.92 mm to (171.8, 100.7)
Connections:
- net /VCC renamed VCC
Routing:
- net VCC: track 0.00 -> 75.0 mm, vias 0 -> 6
- net Net-(D1-Pad2): track 0.00 -> 58.9 mm
- net Net-(D5-Pad2): track 0.00 -> 57.1 mm, vias 0 -> 2
- net Net-(D12-Pad1): track 0.00 -> 47.7 mm
- net Net-(D10-Pad2): track 0.00 -> 43.8 mm, vias 0 -> 4
- net /RST: track 0.00 -> 38.6 mm, vias 0 -> 2
- net Net-(D1-Pad1): track 0.00 -> 31.6 mm, vias 0 -> 4
- net Net-(D10-Pad1): track 0.00 -> 28.2 mm, vias 0 -> 2
- net Net-(D13-Pad1): track 0.00 -> 24.5 mm, vias 0 -> 2
- net Net-(D11-Pad1): track 0.00 -> 21.2 mm
- net Net-(R5-Pad2): track 0.00 -> 21.0 mm, vias 0 -> 2
- net Net-(SW1-Pad1): track 0.00 -> 18.1 mm, vias 0 -> 1
- net Net-(J1-Pad2): track 0.00 -> 17.3 mm, vias 0 -> 1
- net Net-(J1-Pad3): track 0.00 -> 17.2 mm, vias 0 -> 1
- net /MOSI: track 0.00 -> 16.5 mm, vias 0 -> 1
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